File: pico-datalogger-v3.kicad_sch (KiCad schematic)
At the start: 38 parts, among them IC1 LM66200DRLR, J1 JST-PH2 Bat, J11 Conn_I2C1, J12 Conn_UART_5V, J13 THT_I2C1, J14 THT_I2C0, J17 Disp_THT, J2 Conn_Pico_Left, J3 Conn_Pico_Right, J4 SM06B-GHS-TB_LF_SN, J6 Conn_Display, J9 Conn_I2C0, Q1 AO3401A, Q2 AO3401A, U1 74LVC2G74, U2 PCF8523T, U3 Pico, U4 XTSD, Y1 Crystal

Commit message: fix pin-order for SEN66-connector
Connections:
- net +3V3: now also J4.6
- net GND: now also J4.5
- net SCL: now also J4.3; no longer J4.4
- net SDA: now also J4.4; no longer J4.3
- no-connect marks 13 -> 11
Other:
- note added: "Pin-Layout is for JST-GH6 cables with "opposite side" connectors, e.g. Adafruit 5754"
- note added: "SEN66 Connector"
- moved on the sheet: J4
Changed lines of the file:
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@@
   (title_block
     (title "pico-datalogger-v3")
-    (date "2025-11-10")
+    (date "2025-11-12")
     (rev "3.00")
     (company "Bernhard Bablok")
@@
   (junction (at 93.98 72.39) (diameter 0) (color 0 0 0 0)
   )
-  (junction (at 130.81 158.75) (diameter 0) (color 0 0 0 0)
+  (junction (at 166.37 161.29) (diameter 0) (color 0 0 0 0)
   )
   (junction (at 168.91 119.38) (diameter 0) (color 0 0 0 0)
@@
   (no_connect (at 241.3 152.4))
   (no_connect (at 86.36 127))
-  (no_connect (at 133.35 151.13))
   (no_connect (at 76.2 82.55))
   (no_connect (at 91.44 41.91))
@@
   (no_connect (at 231.14 92.71))
   (no_connect (at 86.36 132.08))
-  (no_connect (at 133.35 153.67))
   (no_connect (at 241.3 149.86))
   (wire (pts (xy 133.35 40.64) (xy 134.62 40.64))
@@
     (stroke (width 0) (type default))
   )
-  (wire (pts (xy 130.81 158.75) (xy 133.35 158.75))
+  (wire (pts (xy 166.37 161.29) (xy 168.91 161.29))
     (stroke (width 0) (type default))
   )
@@
     (stroke (width 0) (type default))
   )
-  (wire (pts (xy 130.81 156.21) (xy 130.81 158.75))
+  (wire (pts (xy 166.37 158.75) (xy 166.37 161.29))
     (stroke (width 0) (type default))
   )
@@
     (stroke (width 0) (type default))
   )
-  (wire (pts (xy 124.46 158.75) (xy 130.81 158.75))
+  (wire (pts (xy 160.02 161.29) (xy 166.37 161.29))
     (stroke (width 0) (type default))
   )
@@
     (stroke (width 0) (type default))
   )
-  (wire (pts (xy 133.35 156.21) (xy 130.81 156.21))
+  (wire (pts (xy 168.91 158.75) (xy 166.37 158.75))
     (stroke (width 0) (type default))
   )
@@
     (stroke (width 0) (type default))
   )
+  (rectangle (start 115.57 134.62) (end 195.58 165.1)
+    (stroke (width 0) (type dash))
+    (fill (type none))
+  )
   (image (at 276.86 173.736) (scale 0.540354)
     (data
@@
     (effects (font (size 1.27 1.27)) (justify left bottom))
   )
+  (text "SEN66 Connector" (at 116.84 163.83 0)
+    (effects (font (size 1.27 1.27)) (justify left bottom))
+  )
   (text "RTC: on: high->low" (at 117.094 60.96 0)
     (effects (font (size 1.27 1.27)) (justify left bottom))
@@
     (effects (font (size 1.27 1.27)) (justify left bottom))
   )
+  (text "Pin-Layout is for JST-GH6 cables\nwith \"opposite side\" connectors,\ne.g. Adafruit 5754"
+    (at 116.84 142.24 0)
+    (effects (font (size 1.27 1.27)) (justify left bottom))
+  )
   (text "Connectors (I2C)" (at 116.586 98.806 0)
     (effects (font (size 1.27 1.27)) (justify left bottom))
@@
     )
   )
-  (global_label "SDA" (shape bidirectional) (at 133.35 146.05 180) (fields_autoplaced)
+  (global_label "SDA" (shape bidirectional) (at 168.91 151.13 180) (fields_autoplaced)
     (effects (font (size 1.27 1.27)) (justify right))
-    (property "Intersheetrefs" "${INTERSHEET_REFS}" (at 126.4984 146.05 0)
+    (property "Intersheetrefs" "${INTERSHEET_REFS}" (at 162.0584 151.13 0)
       (effects (font (size 1.27 1.27)) (justify right) hide)
     )
@@
     )
   )
-  (global_label "SCL" (shape bidirectional) (at 133.35 148.59 180) (fields_autoplaced)
+  (global_label "SCL" (shape bidirectional) (at 168.91 148.59 180) (fields_autoplaced)
     (effects (font (size 1.27 1.27)) (justify right))
-    (property "Intersheetrefs" "${INTERSHEET_REFS}" (at 126.5589 148.59 0)
+    (property "Intersheetrefs" "${INTERSHEET_REFS}" (at 162.1189 148.59 0)
       (effects (font (size 1.27 1.27)) (justify right) hide)
     )
@@
     )
   )
-  (symbol (lib_id "power:GND") (at 124.46 158.75 270) (unit 1)
+  (symbol (lib_id "power:GND") (at 160.02 161.29 270) (unit 1)
     (in_bom yes) (on_board yes) (dnp no)
-    (property "Reference" "#PWR08" (at 118.11 158.75 0)
+    (property "Reference" "#PWR08" (at 153.67 161.29 0)
       (effects (font (size 1.27 1.27)) hide)
     )
-    (property "Value" "GND" (at 117.602 158.75 90)
+    (property "Value" "GND" (at 153.162 161.29 90)
       (effects (font (size 1.27 1.27)) (justify left))
     )
-    (property "Footprint" "" (at 124.46 158.75 0)
+    (property "Footprint" "" (at 160.02 161.29 0)
       (effects (font (size 1.27 1.27)) hide)
     )
-    (property "Datasheet" "" (at 124.46 158.75 0)
+    (property "Datasheet" "" (at 160.02 161.29 0)
       (effects (font (size 1.27 1.27)) hide)
     )
@@
     )
   )
-  (symbol (lib_id "power:+3V3") (at 133.35 140.97 90) (unit 1)
+  (symbol (lib_id "power:+3V3") (at 168.91 143.51 90) (unit 1)
     (in_bom yes) (on_board yes) (dnp no)
-    (property "Reference" "#PWR041" (at 137.16 140.97 0)
+    (property "Reference" "#PWR041" (at 172.72 143.51 0)
       (effects (font (size 1.27 1.27)) hide)
     )
-    (property "Value" "+3V3" (at 125.222 140.97 90)
+    (property "Value" "+3V3" (at 160.782 143.51 90)
       (effects (font (size 1.27 1.27)) (justify right))
     )
-    (property "Footprint" "" (at 133.35 140.97 0)
+    (property "Footprint" "" (at 168.91 143.51 0)
       (effects (font (size 1.27 1.27)) hide)
     )
-    (property "Datasheet" "" (at 133.35 140.97 0)
+    (property "Datasheet" "" (at 168.91 143.51 0)
       (effects (font (size 1.27 1.27)) hide)
     )
@@
     )
   )
+  (symbol (lib_id "power:+3V3") (at 168.91 156.21 90) (unit 1)
+    (in_bom yes) (on_board yes) (dnp no)
+    (property "Reference" "#PWR045" (at 172.72 156.21 0)
+      (effects (font (size 1.27 1.27)) hide)
+    )
+    (property "Value" "+3V3" (at 160.782 156.21 90)
+      (effects (font (size 1.27 1.27)) (justify right))
+    )
+    (property "Footprint" "" (at 168.91 156.21 0)
+      (effects (font (size 1.27 1.27)) hide)
+    )
+    (property "Datasheet" "" (at 168.91 156.21 0)
+      (effects (font (size 1.27 1.27)) hide)
+    )
+    (pin "1")
+    (instances
+      (project "pico-datalogger-v3"
+        (path "/17133424-0baa-43c4-a5ff-fd6573e84d8e"
+          (reference "#PWR045") (unit 1)
+        )
+      )
+    )
+  )
   (symbol (lib_id "power:GND") (at 156.21 55.88 0) (unit 1)
     (in_bom yes) (on_board yes) (dnp no) (fields_autoplaced)
@@
     )
   )
-  (symbol (lib_id "user:SM06B-GHS-TB_LF__SN_") (at 143.51 148.59 0) (unit 1)
+  (symbol (lib_id "user:SM06B-GHS-TB_LF__SN_") (at 179.07 151.13 0) (unit 1)
     (in_bom yes) (on_board yes) (dnp no)
-    (property "Reference" "J4" (at 142.24 134.62 0)
+    (property "Reference" "J4" (at 177.8 137.16 0)
       (effects (font (size 1.27 1.27)) (justify left))
     )
-    (property "Value" "SM06B-GHS-TB_LF_SN" (at 133.35 137.16 0)
+    (property "Value" "SM06B-GHS-TB_LF_SN" (at 168.91 139.7 0)
       (effects (font (size 1.27 1.27)) (justify left))
     )
-    (property "Footprint" "user:JST_SM06B-GHS-TB_LF_SN" (at 146.05 167.64 0)
+    (property "Footprint" "user:JST_SM06B-GHS-TB_LF_SN" (at 181.61 170.18 0)
       (effects (font (size 1.27 1.27)) (justify bottom) hide)
     )
-    (property "Datasheet" "" (at 143.51 148.59 0)
+    (property "Datasheet" "" (at 179.07 151.13 0)
       (effects (font (size 1.27 1.27)) hide)
     )
-    (property "MAXIMUM_PACKAGE_HEIGHT" "4.25mm" (at 143.51 175.26 0)
+    (property "MAXIMUM_PACKAGE_HEIGHT" "4.25mm" (at 179.07 177.8 0)
       (effects (font (size 1.27 1.27)) (justify bottom) hide)
     )
-    (property "Description" "Connector Header Surface Mount, Right Angle 6 position 0.049 (1.25mm)" (at 147.32 171.45 0)
+    (property "Description" "Connector Header Surface Mount, Right Angle 6 position 0.049 (1.25mm)" (at 182.88 173.99 0)
       (effects (font (size 1.27 1.27)) (justify bottom) hide)
     )
-    (property "LCSC" "C133065" (at 143.51 148.59 0)
+    (property "LCSC" "C133065" (at 179.07 151.13 0)
       (effects (font (size 1.27 1.27)) hide)
     )
@@
     )
   )
-  (symbol (lib_id "power:GND") (at 133.35 143.51 270) (unit 1)
+  (symbol (lib_id "power:GND") (at 168.91 146.05 270) (unit 1)
     (in_bom yes) (on_board yes) (dnp no)
-    (property "Reference" "#PWR040" (at 127 143.51 0)
+    (property "Reference" "#PWR040" (at 162.56 146.05 0)
       (effects (font (size 1.27 1.27)) hide)
     )
-    (property "Value" "GND" (at 126.492 143.51 90)
+    (property "Value" "GND" (at 162.052 146.05 90)
       (effects (font (size 1.27 1.27)) (justify left))
     )
-    (property "Footprint" "" (at 133.35 143.51 0)
+    (property "Footprint" "" (at 168.91 146.05 0)
       (effects (font (size 1.27 1.27)) hide)
     )
-    (property "Datasheet" "" (at 133.35 143.51 0)
+    (property "Datasheet" "" (at 168.91 146.05 0)
       (effects (font (size 1.27 1.27)) hide)
     )
@@
         )
       )
+    )
+  )
+  (symbol (lib_id "power:GND") (at 168.91 153.67 270) (unit 1)
+    (in_bom yes) (on_board yes) (dnp no)
+    (property "Reference" "#PWR046" (at 162.56 153.67 0)
+      (effects (font (size 1.27 1.27)) hide)
+    )
+    (property "Value" "GND" (at 162.052 153.67 90)
+      (effects (font (size 1.27 1.27)) (justify left))
+    )
+    (property "Footprint" "" (at 168.91 153.67 0)
+      (effects (font (size 1.27 1.27)) hide)
+    )
+    (property "Datasheet" "" (at 168.91 153.67 0)
+      (effects (font (size 1.27 1.27)) hide)
+    )
+    (pin "1")
+    (instances
+      (project "pico-datalogger-v3"
+        (path "/17133424-0baa-43c4-a5ff-fd6573e84d8e"
+          (reference "#PWR046") (unit 1)
+        )
+      )

Commit message: switch to user:JST-PH2
Parts:
- J1: footprint Connector_JST:JST_PH_S2B-PH-SM4-TB_1x02-1MP_P2.00mm_Horizontal -> user:JST_PH_S2B-PH-SM4-TB_1x02-1MP_P2.00mm_Horizontal
Changed lines of the file:
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@@
       (effects (font (size 1.27 1.27)))
     )
-    (property "Footprint" "Connector_JST:JST_PH_S2B-PH-SM4-TB_1x02-1MP_P2.00mm_Horizontal" (at 208.28 77.47 0)
+    (property "Footprint" "user:JST_PH_S2B-PH-SM4-TB_1x02-1MP_P2.00mm_Horizontal" (at 208.28 77.47 0)
       (effects (font (size 1.27 1.27)) hide)
     )

Commit message: switch to user:JST-SH4
Parts:
- J11, J9: footprint Connector_JST:JST_SH_SM04B-SRSS-TB_1x04-1MP_P1.00mm_Horizontal -> user:JST_SH_SM04B-SRSS-TB_1x04-1MP_P1.00mm_Horizontal
Changed lines of the file:
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@@
       (effects (font (size 1.27 1.27)) (justify left))
     )
-    (property "Footprint" "Connector_JST:JST_SH_SM04B-SRSS-TB_1x04-1MP_P1.00mm_Horizontal" (at 124.46 88.9 0)
+    (property "Footprint" "user:JST_SH_SM04B-SRSS-TB_1x04-1MP_P1.00mm_Horizontal" (at 124.46 88.9 0)
       (effects (font (size 1.27 1.27)) hide)
     )
@@
       (effects (font (size 1.27 1.27)) (justify left))
     )
-    (property "Footprint" "Connector_JST:JST_SH_SM04B-SRSS-TB_1x04-1MP_P1.00mm_Horizontal" (at 123.19 72.39 0)
-      (effects (font (size 1.27 1.27)) hide)
-    )
+    (property "Footprint" "user:JST_SH_SM04B-SRSS-TB_1x04-1MP_P1.00mm_Horizontal" (at 123.19 72.39 0)
+      (effects (font (size 1.27 1.27)) hide)
+    )

Commit message: switch to user:JST_SUR_BM08B-SURS-TF_1x08-1MP_P0.80mm_Vertical
Parts:
- J6: footprint Connector_JST:JST_SUR_BM08B-SURS-TF_1x08-1MP_P0.80mm_Vertical -> user:JST_SUR_BM08B-SURS-TF_1x08-1MP_P0.80mm_Vertical; symbol Connector_Generic:Conn_01x08 -> user:JST_SURS08_Vertical
Changed lines of the file:
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@@
     )
   )
-  (symbol (lib_id "Connector_Generic:Conn_01x08") (at 173.99 119.38 0) (mirror x) (unit 1)
+  (symbol (lib_id "user:JST_SURS08_Vertical") (at 173.99 119.38 0) (mirror x) (unit 1)
     (in_bom yes) (on_board yes) (dnp no)
     (property "Reference" "J6" (at 172.72 104.14 0)
@@
       (effects (font (size 1.27 1.27)) (justify left))
     )
-    (property "Footprint" "Connector_JST:JST_SUR_BM08B-SURS-TF_1x08-1MP_P0.80mm_Vertical" (at 173.99 119.38 0)
+    (property "Footprint" "user:JST_SUR_BM08B-SURS-TF_1x08-1MP_P0.80mm_Vertical" (at 173.99 104.14 0)
       (effects (font (size 1.27 1.27)) hide)
     )

Commit message: connect status-pin of diode to GP28
Connections:
- net PDM_DAT is gone; now on net PS_STATUS: J3.7 (Pin_7), U3.34 (GPIO28_ADC2)
- net PS_STATUS: now reaches IC1.8 (ST)
- no-connect marks 11 -> 10
Changed lines of the file:
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@@
   (title_block
     (title "pico-datalogger-v3")
-    (date "2025-11-12")
+    (date "2025-11-18")
     (rev "3.00")
     (company "Bernhard Bablok")
@@
   (no_connect (at 76.2 82.55))
   (no_connect (at 91.44 41.91))
-  (no_connect (at 256.54 72.39))
   (no_connect (at 205.74 92.71))
   (no_connect (at 71.12 82.55))
@@
   (polyline (pts (xy 115.316 17.653) (xy 115.57 62.23))
     (stroke (width 0) (type dash))
+  )
+  (wire (pts (xy 256.54 66.04) (xy 256.54 72.39))
+    (stroke (width 0) (type default))
   )
   (polyline (pts (xy 39.878 108.712) (xy 113.03 108.712))
@@
     (effects (font (size 1.27 1.27)) (justify left bottom))
   )
-  (label "PDM_DAT" (at 95.25 134.62 0) (fields_autoplaced)
-    (effects (font (size 1.27 1.27)) (justify left bottom))
-  )
   (label "PC_GATE" (at 264.16 111.76 0) (fields_autoplaced)
     (effects (font (size 1.27 1.27)) (justify left bottom))
   )
+  (label "PS_STATUS" (at 95.25 134.62 0) (fields_autoplaced)
+    (effects (font (size 1.27 1.27)) (justify left bottom))
+  )
   (label "RX" (at 163.83 95.25 0) (fields_autoplaced)
     (effects (font (size 1.27 1.27)) (justify left bottom))
@@
     (effects (font (size 1.27 1.27)) (justify left bottom))
   )
+  (label "PS_STATUS" (at 256.54 66.04 0) (fields_autoplaced)
+    (effects (font (size 1.27 1.27)) (justify left bottom))
+  )
   (label "SWA" (at 54.61 142.24 180) (fields_autoplaced)
     (effects (font (size 1.27 1.27)) (justify right bottom))
@@
     (effects (font (size 1.27 1.27)) (justify left bottom))
   )
-  (label "PDM_DAT" (at 99.06 44.45 0) (fields_autoplaced)
-    (effects (font (size 1.27 1.27)) (justify left bottom))
-  )
+  (label "PS_STATUS" (at 99.06 44.45 0) (fields_autoplaced)
+    (effects (font (size 1.27 1.27)) (justify left bottom))
+  )

Commit message: swapped SWA/SWB with LoRa-RST/LoRa-CS; initial routing of LoRa and buttons
Parts:
- Y1: footprint Crystal:Crystal_SMD_3215-2Pin_3.2x1.5mm -> user:Crystal_SMD_3215-2Pin_3.2x1.5mm
Connections:
- net Lora_CS: now also J2.12 (Pin_12), U3.12 (GPIO9); no longer J2.17 (Pin_17), U3.17 (GPIO13)
- net Lora_RST: now also J2.10 (Pin_10), U3.10 (GPIO7); no longer J2.16 (Pin_16), U3.16 (GPIO12)
- net SWA: now also J2.16 (Pin_16), U3.16 (GPIO12); no longer J2.10 (Pin_10), U3.10 (GPIO7)
- net SWB: now also J2.17 (Pin_17), U3.17 (GPIO13); no longer J2.12 (Pin_12), U3.12 (GPIO9)
- net PDM_CLK: no longer names the net of J2.7 (Pin_7)
- net PDM_CLK: no longer U3.7 (GPIO5)
- no-connect marks 10 -> 12

Commit message: swapped additional pins to simplify routing
Connections:
- net MISO1: now also J2.16 (Pin_16), U3.16 (GPIO12); no longer J2.11 (Pin_11), U3.11 (GPIO8)
- net SWA: now also J2.11 (Pin_11), U3.11 (GPIO8); no longer J2.16 (Pin_16), U3.16 (GPIO12)
- net SWB: now also J2.9 (Pin_9), U3.9 (GPIO6); no longer J2.17 (Pin_17), U3.17 (GPIO13)
- net SWC: now also J2.17 (Pin_17), U3.17 (GPIO13); no longer J2.19 (Pin_19), U3.19 (GPIO14)
- net SWD: now also J2.7 (Pin_7), U3.7 (GPIO5); no longer J2.9 (Pin_9), U3.9 (GPIO6)

Commit message: fixes for production files
Parts:
- BT2: footprint Battery:BatteryHolder_Keystone_2462_2xAA -> user:BatteryHolder_Keystone_2462_2xAA
Changed lines of the file:
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@@
   (title_block
     (title "pico-datalogger-v3")
-    (date "2025-11-20")
+    (date "2025-11-21")
     (rev "3.00")
     (company "Bernhard Bablok")
@@
       (effects (font (size 1.27 1.27)) (justify left))
     )
-    (property "Footprint" "Battery:BatteryHolder_Keystone_2462_2xAA" (at 269.24 73.406 90)
+    (property "Footprint" "user:BatteryHolder_Keystone_2462_2xAA" (at 269.24 73.406 90)
       (effects (font (size 1.27 1.27)) hide)
     )
