File: lora.kicad_sch (KiCad schematic)
At the start: 4 parts, among them U7 RFM95W-868S2

Commit message: updated production-files for datalogger-v3 (with rfm95-868)
Parts:
- U7: LCSC C2844474 -> C2844472
Changed lines of the file:
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@@
       (effects (font (size 1.27 1.27)) hide)
     )
-    (property "LCSC" "C2844474" (at 66.04 46.99 0)
+    (property "LCSC" "C2844472" (at 66.04 46.99 0)
       (effects (font (size 1.27 1.27)) hide)
     )
